Commit message: fix(sim): align /control mapping and E-Stop with real D-Racer
Invert steering for Gazebo (+right), send steer angle instead of yaw rate, latch E-Stop in the control bridge, and document the shared control contract.

Co-authored-by: Cursor <cursoragent@cursor.com>

File: src/dracer_sim/urdf/dracer_sim.urdf (robot description, URDF)
Before this commit: robot dracer_sim, 5 links, 4 joints
Joints:
- joint camera_joint: origin xyz=0.10 0 0.03 rpy=0 0.25 0 -> xyz=0.10 0 0.08 rpy=0 0.174533 0
