Commit message: feat(control,lane): mask corridor follow, sign-gated OUT forks, lean viz
Add mask_p NORMAL tracker with course-color corridor and fork-force PP,
arm OUT fork perception only after a turn sign, collapse OpenCV to Lane
drive (+HSV), and ship IN/OUT lap and mask-policy benches for A/B.

Co-authored-by: Cursor <cursoragent@cursor.com>

File: vendor/limo_car/gazebo/ackermann.xacro (robot description, xacro)
@@ -79,6 +79,6 @@
             <axis xyz="0 0 1" />
             <!-- Paramenten von Herstellern -->
-            <limit lower="-0.523598767" upper="0.523598767" effort="5" velocity="0.5" />
-            <dynamics damping="1.0" friction="2.0"/>
+            <limit lower="-0.523598767" upper="0.523598767" effort="20" velocity="4.0" />
+            <dynamics damping="0.05" friction="0.05"/>
         </joint>
         <transmission name="${wheel_prefix}_hinge_trans" type="SimpleTransmission">
@@ -151,6 +151,6 @@
             <xacro:insert_block name="joint_pose"/>
             <axis xyz="0 0 -1"/>
-            <limit lower="-0.523598767" upper="0.523598767" effort="5" velocity="0.5" />
-            <dynamics damping="1.0" friction="2.0"/>
+            <limit lower="-0.523598767" upper="0.523598767" effort="20" velocity="4.0" />
+            <dynamics damping="0.05" friction="0.05"/>
         </joint>
         <transmission name="${wheel_prefix}_hinge_trans" type="SimpleTransmission">

File: vendor/limo_car/urdf/limo_steering_hinge.xacro (robot description, xacro)
@@ -31,6 +31,8 @@
             <xacro:insert_block name="joint_pose"/>
             <axis xyz="0 0 1" />
-            <limit lower="-0.523598767" upper="0.523598767" effort="5" velocity="0.5" />
-            <dynamics damping="1.0" friction="2.0"/>
+            <!-- Default vendor 0.5 rad/s felt like slow servo lag; raise for responsive
+                 lane following (~full lock ~0.13 s). -->
+            <limit lower="-0.523598767" upper="0.523598767" effort="20" velocity="4.0" />
+            <dynamics damping="0.05" friction="0.05"/>
         </joint>
         <link name="front_left_wheel_link">
@@ -85,6 +87,6 @@
             <xacro:insert_block name="joint_pose"/>
             <axis xyz="0 0 -1"/>
-            <limit lower="-0.523598767" upper="0.523598767" effort="5" velocity="0.5" />
-            <dynamics damping="1.0" friction="2.0"/>
+            <limit lower="-0.523598767" upper="0.523598767" effort="20" velocity="4.0" />
+            <dynamics damping="0.05" friction="0.05"/>
         </joint>
         <link name="front_right_wheel_link">

Commit message: freeze(control): board-ready low-speed mask_hard_wide with fork L/R verify
Lock NORMAL to mask_p + white hard corridor (cruise 0.28) and align δ_max
to R_min geometry so this branch can ship to the car. Keep fork branch PP,
live spawn visual checks, and tuner/bench harnesses for real-car tuning.

Co-authored-by: Cursor <cursoragent@cursor.com>

File: vendor/limo_car/gazebo/ackermann.xacro (robot description, xacro)
@@ -79,5 +79,6 @@
             <axis xyz="0 0 1" />
             <!-- Paramenten von Herstellern -->
-            <limit lower="-0.523598767" upper="0.523598767" effort="20" velocity="4.0" />
+            <!-- R_min=0.385 m @ L=0.24 → ±atan(L/R)≈0.5574 rad; vel ≈ full-lock ~70 ms -->
+            <limit lower="-0.5574" upper="0.5574" effort="20" velocity="8.0" />
             <dynamics damping="0.05" friction="0.05"/>
         </joint>
@@ -151,5 +152,6 @@
             <xacro:insert_block name="joint_pose"/>
             <axis xyz="0 0 -1"/>
-            <limit lower="-0.523598767" upper="0.523598767" effort="20" velocity="4.0" />
+            <!-- R_min=0.385 m @ L=0.24 → ±atan(L/R)≈0.5574 rad; vel ≈ full-lock ~70 ms -->
+            <limit lower="-0.5574" upper="0.5574" effort="20" velocity="8.0" />
             <dynamics damping="0.05" friction="0.05"/>
         </joint>
@@ -322,5 +324,5 @@
                 <linear_velocity_pid_gain>0.5 10 0.001</linear_velocity_pid_gain>
                 <linear_velocity_i_range>0 0</linear_velocity_i_range>
-                <max_steer>0.523598767</max_steer>
+                <max_steer>0.5574</max_steer>
                 <wheel_separation>0.172</wheel_separation>
                 <wheel_diameter>0.09</wheel_diameter>

File: vendor/limo_car/urdf/limo_steering_hinge.xacro (robot description, xacro)
@@ -33,5 +33,6 @@
             <!-- Default vendor 0.5 rad/s felt like slow servo lag; raise for responsive
                  lane following (~full lock ~0.13 s). -->
-            <limit lower="-0.523598767" upper="0.523598767" effort="20" velocity="4.0" />
+            <!-- R_min=0.385 m @ L=0.24 → ±atan(L/R)≈0.5574 rad; vel ≈ full-lock ~70 ms -->
+            <limit lower="-0.5574" upper="0.5574" effort="20" velocity="8.0" />
             <dynamics damping="0.05" friction="0.05"/>
         </joint>
@@ -87,5 +88,6 @@
             <xacro:insert_block name="joint_pose"/>
             <axis xyz="0 0 -1"/>
-            <limit lower="-0.523598767" upper="0.523598767" effort="20" velocity="4.0" />
+            <!-- R_min=0.385 m @ L=0.24 → ±atan(L/R)≈0.5574 rad; vel ≈ full-lock ~70 ms -->
+            <limit lower="-0.5574" upper="0.5574" effort="20" velocity="8.0" />
             <dynamics damping="0.05" friction="0.05"/>
         </joint>
